File: caravel-mvp.kicad_pcb (KiCad board)
At the start: 4 copper layers, 39 x 54 mm, 57 parts, among them J1 USB_C_Receptacle_USB2.0, J2 Conn_01x02, J3 Conn_02x04_Odd_Even, J4 Conn_01x06, J5 613012243121, J6 Conn_02x18_Odd_Even, SW1 B3U-1000P, SW2 B3U-1000P, U1 Caravel_QFN, U2 W25Q32JVSS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

Commit message: Reset risetime fix
Parts:
- added C24: 1uF, Capacitor_SMD:C_0603_1608Metric, F.Cu at (100.3, 54.0)
- moved C13 0.37 mm to (100.3, 51.0)
- moved C8 0.37 mm to (100.3, 52.5)
Other:
- board text added: "v1.1"
- board text removed: "v1.0"
Changed lines of the file:
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@@
   (title_block
     (title "Caravel Minimum Viable PCB Sample")
-    (date "2023-09-29")
-    (rev "1.0")
+    (date "2023-10-25")
+    (rev "1.1")
     (company "Psychogenic Technologies INC")
     (comment 1 "(C) 2023 Pat Deegan")
@@
     )
   )
+  (footprint "Capacitor_SMD:C_0603_1608Metric" (layer "F.Cu")
+    (at 100.28 54.02 180)
+    (descr "Capacitor SMD 0603 (1608 Metric), square (rectangular) end terminal, IPC_7351 nominal, (Body size source: IPC-SM-782 page 76, https://www.pcb-3d.com/wordpress/wp-content/uploads/ipc-sm-782a_amendment_1_and_2.pdf), generated with kicad-footprint-generator")
+    (tags "capacitor")
+    (property "JLC" "")
+    (property "MPN" "")
+    (property "Part number" "")
+    (property "Sheetfile" "caravel-mvp.kicad_sch")
+    (property "Sheetname" "")
+    (property "ki_description" "Unpolarized capacitor, small symbol")
+    (property "ki_keywords" "capacitor cap")
+    (attr smd)
+    (fp_text reference "C24" (at 0 -1.43) (layer "F.SilkS")
+        (effects (font (size 0.8 0.8) (thickness 0.15)))
+    )
+    (fp_text value "1uF" (at 0 1.43) (layer "F.Fab")
+        (effects (font (size 1 1) (thickness 0.15)))
+    )
+    (fp_text user "${REFERENCE}" (at 0 0) (layer "F.Fab")
+        (effects (font (size 0.4 0.4) (thickness 0.06)))
+    )
+    (fp_line (start -0.14058 -0.51) (end 0.14058 -0.51)
+      (stroke (width 0.12) (type solid)) (layer "F.SilkS"))
+    (fp_line (start -0.14058 0.51) (end 0.14058 0.51)
+      (stroke (width 0.12) (type solid)) (layer "F.SilkS"))
+    (fp_line (start -1.48 -0.73) (end 1.48 -0.73)
+      (stroke (width 0.05) (type solid)) (layer "F.CrtYd"))
+    (fp_line (start -1.48 0.73) (end -1.48 -0.73)
+      (stroke (width 0.05) (type solid)) (layer "F.CrtYd"))
+    (fp_line (start 1.48 -0.73) (end 1.48 0.73)
+      (stroke (width 0.05) (type solid)) (layer "F.CrtYd"))
+    (fp_line (start 1.48 0.73) (end -1.48 0.73)
+      (stroke (width 0.05) (type solid)) (layer "F.CrtYd"))
+    (fp_line (start -0.8 -0.4) (end 0.8 -0.4)
+      (stroke (width 0.1) (type solid)) (layer "F.Fab"))
+    (fp_line (start -0.8 0.4) (end -0.8 -0.4)
+      (stroke (width 0.1) (type solid)) (layer "F.Fab"))
+    (fp_line (start 0.8 -0.4) (end 0.8 0.4)
+      (stroke (width 0.1) (type solid)) (layer "F.Fab"))
+    (fp_line (start 0.8 0.4) (end -0.8 0.4)
+      (stroke (width 0.1) (type solid)) (layer "F.Fab"))
+    (pad "1" smd roundrect (at -0.775 0 180) (size 0.9 0.95) (layers "F.Cu" "F.Paste" "F.Mask") (roundrect_rratio 0.25)
+      (net 3 "~{SOC_RST}") (pintype "passive"))
+    (pad "2" smd roundrect (at 0.775 0 180) (size 0.9 0.95) (layers "F.Cu" "F.Paste" "F.Mask") (roundrect_rratio 0.25)
+      (net 1 "GND") (pintype "passive"))
+    (model "${KICAD6_3DMODEL_DIR}/Capacitor_SMD.3dshapes/C_0603_1608Metric.wrl"
+      (offset (xyz 0 0 0))
+      (scale (xyz 1 1 1))
+      (rotate (xyz 0 0 0))
+    )
+  )
   (footprint "Resistor_SMD:R_0603_1608Metric" (layer "F.Cu")
     (at 104.2 43.2 90)
@@
   )
   (footprint "Capacitor_SMD:C_0603_1608Metric" (layer "F.Cu")
-    (at 100.62 52.68 180)
+    (at 100.3 52.5 180)
     (descr "Capacitor SMD 0603 (1608 Metric), square (rectangular) end terminal, IPC_7351 nominal, (Body size source: IPC-SM-782 page 76, https://www.pcb-3d.com/wordpress/wp-content/uploads/ipc-sm-782a_amendment_1_and_2.pdf), generated with kicad-footprint-generator")
     (tags "capacitor")
@@
     (property "ki_keywords" "capacitor cap")
     (attr smd)
-    (fp_text reference "C8" (at 0 -1.18) (layer "F.SilkS")
+    (fp_text reference "C8" (at 1.92 -0.02 90) (layer "F.SilkS")
         (effects (font (size 0.8 0.8) (thickness 0.15)))
     )
@@
   )
   (footprint "Capacitor_SMD:C_0603_1608Metric" (layer "F.Cu")
-    (at 100.62 51.18 180)
+    (at 100.3 51 180)
     (descr "Capacitor SMD 0603 (1608 Metric), square (rectangular) end terminal, IPC_7351 nominal, (Body size source: IPC-SM-782 page 76, https://www.pcb-3d.com/wordpress/wp-content/uploads/ipc-sm-782a_amendment_1_and_2.pdf), generated with kicad-footprint-generator")
     (tags "capacitor")
@@
   (gr_arc (start 90 79) (mid 89.292893 78.707107) (end 89 78)
     (stroke (width 0.1) (type default)) (layer "Edge.Cuts"))
-  (gr_text "v1.0" (at 119.7 44.4) (layer "F.SilkS")
+  (gr_text "v1.1" (at 119.7 44.4) (layer "F.SilkS")
     (effects (font (size 1 1) (thickness 0.15)) (justify right bottom))
   )
