File: power_reg.kicad_sch (KiCad schematic)
At the start: 11 parts, among them U2 AZ1117-3.3, U4 AP2112K-1.8

Commit message: Cleanups and even more clarifications in comments
Changed lines of the file:
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@@
   )
   (symbol (lib_id "Device:C_Small") (at 53.34 40.64 0) (unit 1)
-    (in_bom yes) (on_board yes) (dnp no) (fields_autoplaced)
-    (property "Reference" "C8" (at 55.88 39.3762 0)
+    (in_bom yes) (on_board yes) (dnp no)
+    (property "Reference" "C8" (at 49.022 38.862 0)
       (effects (font (size 1.27 1.27)) (justify left))
     )
-    (property "Value" "10uF" (at 55.88 41.9162 0)
+    (property "Value" "10uF" (at 53.34 42.418 0)
       (effects (font (size 1.27 1.27)) (justify left))
     )
@@
   )
   (symbol (lib_id "Device:C_Small") (at 55.88 71.12 0) (unit 1)
-    (in_bom yes) (on_board yes) (dnp no) (fields_autoplaced)
-    (property "Reference" "C9" (at 58.42 69.8562 0)
+    (in_bom yes) (on_board yes) (dnp no)
+    (property "Reference" "C9" (at 51.562 69.596 0)
       (effects (font (size 1.27 1.27)) (justify left))
     )
-    (property "Value" "10uF" (at 58.42 72.3962 0)
+    (property "Value" "10uF" (at 56.134 72.898 0)
       (effects (font (size 1.27 1.27)) (justify left))
     )
